Commit message: Modified the xacro files to make it movable yet awkwardly by directly changing its velocity in the gazebo. Still warning /No pid gain found in /gazebo_ros_control...

File: pan_and_tilt_description/robot/body.xacro (robot description, xacro)
@@ -56,7 +56,7 @@
         <mu1>10.0</mu1>
         <mu2>10.0</mu2>
-        <material>Gazebo/Blue</material>
+        <material>Gazebo/Gray</material>
     </gazebo>
-    <joint name="yaw_joint" type="continuous">
+    <joint name="yaw_joint" type="revolute">
         <parent link="base_link"/>
         <child link="yaw_link"/>
@@ -68,8 +68,8 @@
         <type>transmission_interface/SimpleTransmission</type>
         <joint name="yaw_joint">
-            <hardwareInterface>EffortJointInterface</hardwareInterface>
+            <hardwareInterface>hardware_interface/VelocityJointInterface</hardwareInterface>
         </joint>
         <actuator name="motor1">
-            <hardwareInterface>EffortJointInterface</hardwareInterface>
+            <hardwareInterface>hardware_interface/VelocityJointInterface</hardwareInterface>
             <mechanicalReduction>1</mechanicalReduction>
         </actuator>
@@ -114,8 +114,8 @@
         <type>transmission_interface/SimpleTransmission</type>
         <joint name="pitch_joint">
-            <hardwareInterface>hardware_interface/EffortJointInterface</hardwareInterface>
+            <hardwareInterface>hardware_interface/VelocityJointInterface</hardwareInterface>
         </joint>
         <actuator name="motor2">
-            <hardwareInterface>hardware_interface/EffortJointInterface</hardwareInterface>
+            <hardwareInterface>hardware_interface/VelocityJointInterface</hardwareInterface>
             <mechanicalReduction>1</mechanicalReduction>
         </actuator>

Commit message: Fixed joint position, now it can move correctly. TODO: something wrong with the camera_link rotation, the image is wrong.

File: pan_and_tilt_description/robot/body.xacro (robot description, xacro)
@@ -77,5 +77,5 @@
     <link name="pitch_link">
         <inertial>
-            <origin xyz="0 0 ${BASE_RADIUS*7/5}" rpy="0 ${PI/2} 0"/>
+            <origin xyz="0 0 0" rpy="0 ${PI/2} 0"/>
             <mass value="${joints_mass}" />
             <cylinder_inertia
@@ -91,5 +91,5 @@
         </collision>-->
         <visual>
-            <origin xyz="0 0 ${BASE_RADIUS*7/5}" rpy="0 ${PI/2} 0"/>
+            <origin xyz="0 0 0" rpy="0 ${PI/2} 0"/>
             <geometry>
                 <cylinder radius="${BASE_RADIUS/5*2}" length="${BASE_RADIUS}"/>
@@ -107,5 +107,5 @@
 		<parent link="yaw_link"/>
 		<child link="pitch_link"/>
-		<origin xyz="0.0 0.0 0.0" rpy="0 0 0"/>
+		<origin xyz="0.0 0.0 ${BASE_RADIUS*7/5}" rpy="0 0 0"/>
 		<limit lower="${-85*DEG2RAD}" upper="${85*DEG2RAD}" effort="${joint_pitch_max_effort}" velocity="${joint_pitch_max_speed}"/>
 		<axis xyz="1 0 0"/>
@@ -123,5 +123,5 @@
     <link name="camera_link">
         <inertial>
-            <origin xyz="0 0 0" rpy="0 0 0"/>
+            <origin xyz="${BASE_RADIUS*2/5} 0 0" rpy="0 0 0"/>
             <mass value="0" />
             <mass value="${face_mass}" />
@@ -140,5 +140,5 @@
         </collision>-->
         <visual>
-            <origin xyz="0 0 ${BASE_RADIUS/5*9}" rpy="0 ${-PI/2} 0"/>
+            <origin xyz="${BASE_RADIUS*2/5} 0 0" rpy="0 0 0"/>
             <geometry>
                 <!-- <mesh filename="package://pan_and_tilt_description/meshes/head.stl" scale="1 1 1"/> -->
@@ -157,5 +157,5 @@
 		<parent link="pitch_link"/>
 		<child link="camera_link"/>
-		<origin xyz="0.0 0.0 0.0" rpy="0 0 0"/>
+		<origin xyz="0.0 0.0 0.0" rpy="0 ${-PI/2} 0"/>
 	</joint>
       <!-- camera -->

File: pan_and_tilt_description/robot/pan_and_tilt.xacro (robot description, xacro)
@@ -4,4 +4,5 @@
     <xacro:include filename="$(find pan_and_tilt_description)/robot/common_properties.xacro" />
     <xacro:include filename="$(find pan_and_tilt_description)/robot/body.xacro"/>
+    <!--<xacro:include filename="$(find pan_and_tilt_description)/robot/try.xacro"/>-->
     <body/>
 </robot>

Commit message: Finished camera settings. One camera is done.

File: pan_and_tilt_description/robot/body.xacro (robot description, xacro)
@@ -123,5 +123,5 @@
     <link name="camera_link">
         <inertial>
-            <origin xyz="${BASE_RADIUS*2/5} 0 0" rpy="0 0 0"/>
+            <origin xyz="${BASE_RADIUS/5*2} 0 0 " rpy="0 0 0"/>
             <mass value="0" />
             <mass value="${face_mass}" />
@@ -140,5 +140,5 @@
         </collision>-->
         <visual>
-            <origin xyz="${BASE_RADIUS*2/5} 0 0" rpy="0 0 0"/>
+            <origin xyz="${BASE_RADIUS/5*2} 0 0" rpy="0 0 0"/>
             <geometry>
                 <!-- <mesh filename="package://pan_and_tilt_description/meshes/head.stl" scale="1 1 1"/> -->
@@ -157,8 +157,14 @@
 		<parent link="pitch_link"/>
 		<child link="camera_link"/>
-		<origin xyz="0.0 0.0 0.0" rpy="0 ${-PI/2} 0"/>
+		<origin xyz="0.0 0.0 0.0" rpy="0 ${-PI/2} ${-PI/2}"/>
 	</joint>
+    <link name="vision_link"/>
+    <joint name="vision_camera_joint" type="fixed">
+        <parent link="camera_link"/>
+        <child link="vision_link"/>
+        <origin xyz="${BASE_RADIUS/5*2} 0.0 0.0" rpy="0 0 0"/>
+    </joint>
       <!-- camera -->
-    <gazebo reference="camera_link">
+    <gazebo reference="vision_link">
         <sensor type="camera" name="camera1">
         <update_rate>30.0</update_rate>
@@ -167,6 +173,6 @@
             <horizontal_fov>1.3962634</horizontal_fov>
             <image>
-            <width>400</width>
-            <height>400</height>
+            <width>640</width>
+            <height>480</height>
             <format>R8G8B8</format>
             </image>

Commit message: Get rid of the robot_spawner pkg. TODO: spawn multiple robots

File: pan_and_tilt_description/robot/body.xacro (robot description, xacro)
@@ -108,5 +108,5 @@
 		<child link="pitch_link"/>
 		<origin xyz="0.0 0.0 ${BASE_RADIUS*7/5}" rpy="0 0 0"/>
-		<limit lower="${-85*DEG2RAD}" upper="${85*DEG2RAD}" effort="${joint_pitch_max_effort}" velocity="${joint_pitch_max_speed}"/>
+		<limit lower="${-90*DEG2RAD}" upper="${90*DEG2RAD}" effort="${joint_pitch_max_effort}" velocity="${joint_pitch_max_speed}"/>
 		<axis xyz="1 0 0"/>
 	</joint>

Commit message: 1st advance: change all pan_and_tilt_robot_description to robot_description in all launch files and common_properties.xacro file

File: pan_and_tilt_description/robot/body.xacro (robot description, xacro)
@@ -102,5 +102,5 @@
         <mu1>10.0</mu1>
         <mu2>10.0</mu2>
-        <material>Gazebo/Green</material>
+        <material>Gazebo/Red</material>
     </gazebo>
 	<joint name="pitch_joint" type="revolute">

File: pan_and_tilt_description/robot/common_properties.xacro (robot description, xacro)
@@ -17,5 +17,5 @@
                 filename="libgazebo_ros_control.so">
             <robotNamespace>/pan_and_tilt</robotNamespace>
-            <robotParam>/pan_and_tilt_robot_description</robotParam>
+            <robotParam>/robot_description</robotParam>
             <robotSimType>gazebo_ros_control/DefaultRobotHWSim</robotSimType>
             <legacyModeNS>true</legacyModeNS>

Commit message: main.launch successfully launched a robot with group tag. Ref: https://answers.gazebosim.org//question/16497/spawning-multiple-robots-each-with-a-controller-in-the-same-namespace-as-the-controller_manager/

File: pan_and_tilt_description/robot/body.xacro (robot description, xacro)
@@ -56,5 +56,5 @@
         <mu1>10.0</mu1>
         <mu2>10.0</mu2>
-        <material>Gazebo/Gray</material>
+        <material>Gazebo/Red</material>
     </gazebo>
     <joint name="yaw_joint" type="revolute">
@@ -102,5 +102,5 @@
         <mu1>10.0</mu1>
         <mu2>10.0</mu2>
-        <material>Gazebo/Red</material>
+        <material>Gazebo/Green</material>
     </gazebo>
 	<joint name="pitch_joint" type="revolute">

File: pan_and_tilt_description/robot/common_properties.xacro (robot description, xacro)
@@ -16,6 +16,4 @@
         <plugin name="gazebo_ros_control"
                 filename="libgazebo_ros_control.so">
-            <robotNamespace>/pan_and_tilt</robotNamespace>
-            <robotParam>/robot_description</robotParam>
             <robotSimType>gazebo_ros_control/DefaultRobotHWSim</robotSimType>
             <legacyModeNS>true</legacyModeNS>

Commit message: Modified world light and body.xacro(upper and lower limits of pitch joint)

File: pan_and_tilt_description/robot/body.xacro (robot description, xacro)
@@ -108,5 +108,5 @@
 		<child link="pitch_link"/>
 		<origin xyz="0.0 0.0 ${BASE_RADIUS*7/5}" rpy="0 0 0"/>
-		<limit lower="${-90*DEG2RAD}" upper="${90*DEG2RAD}" effort="${joint_pitch_max_effort}" velocity="${joint_pitch_max_speed}"/>
+		<limit lower="0" upper="${-90*DEG2RAD}" effort="${joint_pitch_max_effort}" velocity="${joint_pitch_max_speed}"/>
 		<axis xyz="1 0 0"/>
 	</joint>
@@ -178,6 +178,6 @@
             </image>
             <clip>
-            <near>0.01</near>
-            <far>10.0</far>
+                <near>0.01</near>
+                <far>200.0</far>
             </clip>
             <noise>

Commit message: Spawn multiple robots in rviz after modified main_sim.launch: added some tf static broadcaster and added two robotModel in rviz panel.

File: pan_and_tilt_description/robot/body.xacro (robot description, xacro)
@@ -24,4 +24,5 @@
         </visual>
     </link>
+    <link name="world"/>
     <joint name="world_base_joint" type="fixed">
         <parent link="world"/>
@@ -108,5 +109,5 @@
 		<child link="pitch_link"/>
 		<origin xyz="0.0 0.0 ${BASE_RADIUS*7/5}" rpy="0 0 0"/>
-		<limit lower="0" upper="${-90*DEG2RAD}" effort="${joint_pitch_max_effort}" velocity="${joint_pitch_max_speed}"/>
+		<limit lower="0" upper="${90*DEG2RAD}" effort="${joint_pitch_max_effort}" velocity="${joint_pitch_max_speed}"/>
 		<axis xyz="1 0 0"/>
 	</joint>

File: pan_and_tilt_description/robot/common_properties.xacro (robot description, xacro)
@@ -12,5 +12,4 @@
     <xacro:property name="BASE_RADIUS" value="0.5" />
     <xacro:property name="INF" value="100000000000000000" />
-    <link name="world"/>
     <gazebo>
         <plugin name="gazebo_ros_control"
